Commit message: Include new model files

File: simulation/spyndra_description/urdf/spyndra.urdf (robot description, URDF)
Before this commit: robot spyndra, 9 links, 8 joints
Joints:
- joint base_to_femur_1: limit lower=-2.0 upper=2.0 effort=50.0 velocity=0.1 -> lower=-1.5 upper=1.5 effort=100.0 velocity=0.1; origin xyz=0.6 0 0.1 rpy=0 0 0 -> xyz=0.9 0 -0.2 rpy=0 0 0
- joint base_to_femur_2: limit lower=-2.0 upper=2.0 effort=50.0 velocity=0.1 -> lower=-1.5 upper=1.5 effort=100.0 velocity=0.1; origin xyz=0 0.6 0.1 rpy=0 0 0 -> xyz=0 0.9 -0.2 rpy=0 0 0
- joint base_to_femur_3: limit lower=-2.0 upper=2.0 effort=50.0 velocity=0.1 -> lower=-1.5 upper=1.5 effort=100.0 velocity=0.1; origin xyz=-0.6 0 0.1 rpy=0 0 0 -> xyz=-0.9 0 -0.2 rpy=0 0 0
- joint base_to_femur_4: limit lower=-2.0 upper=2.0 effort=50.0 velocity=0.1 -> lower=-1.5 upper=1.5 effort=100.0 velocity=0.1; origin xyz=0 -0.6 0.1 rpy=0 0 0 -> xyz=0 -0.9 -0.2 rpy=0 0 0
- joint femur_to_tibia_1: limit lower=-2.0 upper=2.0 effort=50.0 velocity=0.1 -> lower=-1.5 upper=1.5 effort=100.0 velocity=0.1; origin xyz=1.1 0 0 rpy=0 0 0 -> xyz=0.8 0 0 rpy=0 0 0
- joint femur_to_tibia_2: limit lower=-2.0 upper=2.0 effort=50.0 velocity=0.1 -> lower=-1.5 upper=1.5 effort=100.0 velocity=0.1; origin xyz=0 1.1 0 rpy=0 0 0 -> xyz=0 0.8 0 rpy=0 0 0
- joint femur_to_tibia_3: limit lower=-2.0 upper=2.0 effort=50.0 velocity=0.1 -> lower=-1.5 upper=1.5 effort=100.0 velocity=0.1; origin xyz=-1.1 0 0 rpy=0 0 0 -> xyz=-0.8 0 0 rpy=0 0 0
- joint femur_to_tibia_4: limit lower=-2.0 upper=2.0 effort=50.0 velocity=0.1 -> lower=-1.5 upper=1.5 effort=100.0 velocity=0.1; origin xyz=0 -1.1 0 rpy=0 0 0 -> xyz=0 -0.8 0 rpy=0 0 0

Commit message: Fix bugs

File: simulation/spyndra_description/urdf/spyndra.urdf (robot description, URDF)
Before this commit: robot spyndra, 9 links, 8 joints
Joints:
- joint base_to_femur_1: limit lower=-1.5 upper=1.5 effort=100.0 velocity=0.1 -> lower=-1.5 upper=1.5 effort=200.0 velocity=0.1
- joint base_to_femur_2: limit lower=-1.5 upper=1.5 effort=100.0 velocity=0.1 -> lower=-1.5 upper=1.5 effort=200.0 velocity=0.1
- joint base_to_femur_3: limit lower=-1.5 upper=1.5 effort=100.0 velocity=0.1 -> lower=-1.5 upper=1.5 effort=200.0 velocity=0.1
- joint base_to_femur_4: limit lower=-1.5 upper=1.5 effort=100.0 velocity=0.1 -> lower=-1.5 upper=1.5 effort=200.0 velocity=0.1
- joint femur_to_tibia_1: limit lower=-1.5 upper=1.5 effort=100.0 velocity=0.1 -> lower=-1.5 upper=1.5 effort=200.0 velocity=0.1
- joint femur_to_tibia_2: limit lower=-1.5 upper=1.5 effort=100.0 velocity=0.1 -> lower=-1.5 upper=1.5 effort=200.0 velocity=0.1
- joint femur_to_tibia_3: limit lower=-1.5 upper=1.5 effort=100.0 velocity=0.1 -> lower=-1.5 upper=1.5 effort=200.0 velocity=0.1
- joint femur_to_tibia_4: limit lower=-1.5 upper=1.5 effort=100.0 velocity=0.1 -> lower=-1.5 upper=1.5 effort=200.0 velocity=0.1

Commit message: Fix simulation bugs

File: simulation/spyndra_description/urdf/spyndra.urdf (robot description, URDF)
Before this commit: robot spyndra, 9 links, 8 joints
Links:
- link base_link: mass 0.5 -> 1
- link femur_1: mass 0.1 -> 0.2
- link femur_2: mass 0.1 -> 0.2
- link femur_3: mass 0.1 -> 0.2
- link femur_4: mass 0.1 -> 0.2
Joints:
- joint base_to_femur_1: limit lower=-1.5 upper=1.5 effort=200.0 velocity=0.1 -> lower=-1.5 upper=1.5 effort=1000.0 velocity=0.1
- joint base_to_femur_2: limit lower=-1.5 upper=1.5 effort=200.0 velocity=0.1 -> lower=-1.5 upper=1.5 effort=1000.0 velocity=0.1
- joint base_to_femur_3: limit lower=-1.5 upper=1.5 effort=200.0 velocity=0.1 -> lower=-1.5 upper=1.5 effort=1000.0 velocity=0.1
- joint base_to_femur_4: limit lower=-1.5 upper=1.5 effort=200.0 velocity=0.1 -> lower=-1.5 upper=1.5 effort=1000.0 velocity=0.1
- joint femur_to_tibia_1: limit lower=-1.5 upper=1.5 effort=200.0 velocity=0.1 -> lower=-1.5 upper=1.5 effort=1000.0 velocity=0.1
- joint femur_to_tibia_2: limit lower=-1.5 upper=1.5 effort=200.0 velocity=0.1 -> lower=-1.5 upper=1.5 effort=1000.0 velocity=0.1
- joint femur_to_tibia_3: limit lower=-1.5 upper=1.5 effort=200.0 velocity=0.1 -> lower=-1.5 upper=1.5 effort=1000.0 velocity=0.1
- joint femur_to_tibia_4: limit lower=-1.5 upper=1.5 effort=200.0 velocity=0.1 -> lower=-1.5 upper=1.5 effort=1000.0 velocity=0.1

Commit message: Fix robot sliding and position noise issues

File: simulation/spyndra_description/urdf/spyndra.urdf (robot description, URDF)
Before this commit: robot spyndra, 9 links, 8 joints
Joints:
- joint base_to_femur_1: limit lower=-1.5 upper=1.5 effort=1000.0 velocity=0.1 -> lower=-3 upper=3 effort=1000.0 velocity=1
- joint base_to_femur_2: limit lower=-1.5 upper=1.5 effort=1000.0 velocity=0.1 -> lower=-3 upper=3 effort=1000.0 velocity=1
- joint base_to_femur_3: limit lower=-1.5 upper=1.5 effort=1000.0 velocity=0.1 -> lower=-3 upper=3 effort=1000.0 velocity=1
- joint base_to_femur_4: limit lower=-1.5 upper=1.5 effort=1000.0 velocity=0.1 -> lower=-3 upper=3 effort=1000.0 velocity=1
- joint femur_to_tibia_1: limit lower=-1.5 upper=1.5 effort=1000.0 velocity=0.1 -> lower=-3 upper=3 effort=1000.0 velocity=1
- joint femur_to_tibia_2: limit lower=-1.5 upper=1.5 effort=1000.0 velocity=0.1 -> lower=-3 upper=3 effort=1000.0 velocity=1
- joint femur_to_tibia_3: limit lower=-1.5 upper=1.5 effort=1000.0 velocity=0.1 -> lower=-3 upper=3 effort=1000.0 velocity=1
- joint femur_to_tibia_4: limit lower=-1.5 upper=1.5 effort=1000.0 velocity=0.1 -> lower=-3 upper=3 effort=1000.0 velocity=1
